Commit message: Added Controller file and ros2_control also simulated robot in rviz only

File: robotic_arm/urdf/robotic.xacro (robot description, xacro)
@@ -2,5 +2,4 @@
 <robot name="robotic" xmlns:xacro="http://www.ros.org/wiki/xacro">
   <xacro:property name="scale" value="0.001 0.001 0.001"/>
-  <xacro:property name="filepath" value="package://robotic_arm//meshes"/>
   <material name="silver">
     <color rgba="0.700 0.700 0.700 1.000"/>
@@ -14,5 +13,5 @@
     <visual>
       <geometry>
-        <mesh filename="${filepath}/base_link.stl" scale="${scale}"/>
+        <mesh filename="package://robotic_arm/meshes/base_link.stl" scale="${scale}"/>
       </geometry>
       <origin xyz="0 0 0" rpy="0 0 0"/>
@@ -21,5 +20,5 @@
     <collision>
       <geometry>
-        <mesh filename="${filepath}/base_link.stl" scale="${scale}"/>
+        <mesh filename="package://robotic_arm/meshes/base_link.stl" scale="${scale}"/>
       </geometry>
       <origin xyz="0 0 0" rpy="0 0 0"/>
@@ -35,5 +34,5 @@
       <origin xyz="-0.0 -0.0 -0.029" rpy="0 0 0"/>
       <geometry>
-        <mesh filename="${filepath}/Link_1_1.stl" scale="${scale}"/>
+        <mesh filename="package://robotic_arm/meshes/Link_1_1.stl" scale="${scale}"/>
       </geometry>
       <material name="silver"/>
@@ -42,5 +41,5 @@
       <origin xyz="-0.0 -0.0 -0.029" rpy="0 0 0"/>
       <geometry>
-        <mesh filename="${filepath}/Link_1_1.stl" scale="${scale}"/>
+        <mesh filename="package://robotic_arm/meshes/Link_1_1.stl" scale="${scale}"/>
       </geometry>
     </collision>
@@ -55,5 +54,5 @@
       <origin xyz="0.016725 -0.044458 -0.249" rpy="0 0 0"/>
       <geometry>
-        <mesh filename="${filepath}/link_2_1.stl" scale="${scale}"/>
+        <mesh filename="package://robotic_arm/meshes/link_2_1.stl" scale="${scale}"/>
       </geometry>
       <material name="silver"/>
@@ -62,5 +61,5 @@
       <origin xyz="0.016725 -0.044458 -0.249" rpy="0 0 0"/>
       <geometry>
-        <mesh filename="${filepath}/link_2_1.stl" scale="${scale}"/>
+        <mesh filename="package://robotic_arm/meshes/link_2_1.stl" scale="${scale}"/>
       </geometry>
     </collision>
@@ -75,5 +74,5 @@
       <origin xyz="0.15096 0.021534 -0.267342" rpy="0 0 0"/>
       <geometry>
-        <mesh filename="${filepath}/link3_part_1.stl" scale="${scale}"/>
+        <mesh filename="package://robotic_arm/meshes/link3_part_1.stl" scale="${scale}"/>
       </geometry>
       <material name="silver"/>
@@ -82,9 +81,9 @@
       <origin xyz="0.15096 0.021534 -0.267342" rpy="0 0 0"/>
       <geometry>
-        <mesh filename="${filepath}/link3_part_1.stl" scale="${scale}"/>
+        <mesh filename="package://robotic_arm/meshes/link3_part_1.stl" scale="${scale}"/>
       </geometry>
     </collision>
   </link>
-  <joint name="Revolute 1" type="continuous">
+  <joint name="Revolute_1" type="continuous">
     <origin xyz="0.0 0.0 0.029" rpy="0 0 0"/>
     <parent link="base_link"/>
@@ -92,5 +91,5 @@
     <axis xyz="0.0 0.0 1.0"/>
   </joint>
-  <joint name="Revolute 2" type="revolute">
+  <joint name="Revolute_2" type="revolute">
     <origin xyz="-0.016725 0.044458 0.22" rpy="0 0 0"/>
     <parent link="Link_1_1"/>
@@ -99,5 +98,5 @@
     <limit upper="1.134464" lower="-4.014257" effort="100" velocity="100"/>
   </joint>
-  <joint name="Revolute 3" type="revolute">
+  <joint name="Revolute_3" type="revolute">
     <origin xyz="-0.134235 -0.065992 0.018342" rpy="0 0 0"/>
     <parent link="link_2_1"/>
@@ -106,3 +105,31 @@
     <limit upper="1.48353" lower="0.0" effort="100" velocity="100"/>
   </joint>
+  <ros2_control name="MockSystem" type="system">
+    <hardware>
+      <plugin>mock_components/GenericSystem</plugin>
+    </hardware>
+    <joint name="Revolute_1">
+      <command_interface name="position"/>
+      <state_interface name="position"/>
+      <state_interface name="velocity"/>
+    </joint>
+    <joint name="Revolute_2">
+      <command_interface name="position"/>
+      <state_interface name="position"/>
+      <state_interface name="velocity"/>
+    </joint>
+    <joint name="Revolute_3">
+      <command_interface name="position"/>
+      <state_interface name="position"/>
+      <state_interface name="velocity"/>
+    </joint>
+  </ros2_control>
 </robot>
+<!--
+Neutral Position of Robotic Arm
+ros2 topic pub /arm_controller/joint_trajectory trajectory_msgs/msg/JointTrajectory "
+joint_names: ['Revolute_1', 'Revolute_2', 'Revolute_3']
+points:
+- positions: [-0.35, 0.2, 0.5]
+  time_from_start: {sec: 2}
+-->

Commit message: Successfully simulated Robot in gazebo, correct launch file and gazebo plugin

File: robotic_arm/urdf/robotic.xacro (robot description, xacro)
@@ -5,4 +5,5 @@
     <color rgba="0.700 0.700 0.700 1.000"/>
   </material>
+  <link name="world"/>
   <link name="base_link">
     <inertial>
@@ -85,4 +86,9 @@
     </collision>
   </link>
+  <joint name="world_base_joint" type="fixed">
+    <origin xyz="0.0 0.0 0.0" rpy="0.0 0.0 0.0"/>
+    <parent link="world"/>
+    <child link="base_link"/>
+  </joint>
   <joint name="Revolute_1" type="continuous">
     <origin xyz="0.0 0.0 0.029" rpy="0 0 0"/>
@@ -90,4 +96,5 @@
     <child link="Link_1_1"/>
     <axis xyz="0.0 0.0 1.0"/>
+    <limit effort="50" velocity="5"/>
   </joint>
   <joint name="Revolute_2" type="revolute">
@@ -96,5 +103,5 @@
     <child link="link_2_1"/>
     <axis xyz="0.352111 -0.935958 -0.0"/>
-    <limit upper="1.134464" lower="-4.014257" effort="100" velocity="100"/>
+    <limit upper="1.134464" lower="-4.014257" effort="50" velocity="5"/>
   </joint>
   <joint name="Revolute_3" type="revolute">
@@ -103,9 +110,16 @@
     <child link="link3_part_1"/>
     <axis xyz="0.352111 -0.935958 -0.0"/>
-    <limit upper="1.48353" lower="0.0" effort="100" velocity="100"/>
+    <limit upper="1.48353" lower="0.0" effort="50" velocity="5"/>
   </joint>
-  <ros2_control name="MockSystem" type="system">
+  <gazebo>
+    <plugin
+      filename="libgz_ros2_control-system.so"
+      name="gz_ros2_control::GazeboSimROS2ControlPlugin">
+      <parameters>$(find robotic_arm)/config/controllers.yaml</parameters>
+    </plugin>
+  </gazebo>
+  <ros2_control name="GazeboSystem" type="system">
     <hardware>
-      <plugin>mock_components/GenericSystem</plugin>
+      <plugin>gz_ros2_control/GazeboSimSystem</plugin>
     </hardware>
     <joint name="Revolute_1">
@@ -132,4 +146,4 @@
 points:
 - positions: [-0.35, 0.2, 0.5]
-  time_from_start: {sec: 2}
+  time_from_start: {sec: 2} "
 -->

Commit message: corrected angles of Arm and changed color

File: robotic_arm/urdf/robotic.xacro (robot description, xacro)
@@ -3,5 +3,5 @@
   <xacro:property name="scale" value="0.001 0.001 0.001"/>
   <material name="silver">
-    <color rgba="0.700 0.700 0.700 1.000"/>
+    <color rgba="0.300 0.300 0.300 1.000"/>
   </material>
   <link name="world"/>
@@ -33,5 +33,5 @@
     </inertial>
     <visual>
-      <origin xyz="-0.0 -0.0 -0.029" rpy="0 0 0"/>
+      <origin xyz="0.0 0.0 -0.1" rpy="0 0 -0.36"/>
       <geometry>
         <mesh filename="package://robotic_arm/meshes/Link_1_1.stl" scale="${scale}"/>
@@ -40,5 +40,5 @@
     </visual>
     <collision>
-      <origin xyz="-0.0 -0.0 -0.029" rpy="0 0 0"/>
+      <origin xyz="0.0 0.0 -0.1" rpy="0 0 -0.36"/>
       <geometry>
         <mesh filename="package://robotic_arm/meshes/Link_1_1.stl" scale="${scale}"/>
@@ -53,5 +53,5 @@
     </inertial>
     <visual>
-      <origin xyz="0.016725 -0.044458 -0.249" rpy="0 0 0"/>
+      <origin xyz="0.000725 -0.044458 -0.249" rpy="0 0 -0.36"/>
       <geometry>
         <mesh filename="package://robotic_arm/meshes/link_2_1.stl" scale="${scale}"/>
@@ -60,5 +60,5 @@
     </visual>
     <collision>
-      <origin xyz="0.016725 -0.044458 -0.249" rpy="0 0 0"/>
+      <origin xyz="0.000725 -0.044458 -0.249" rpy="0 0 -0.36"/>
       <geometry>
         <mesh filename="package://robotic_arm/meshes/link_2_1.stl" scale="${scale}"/>
@@ -73,5 +73,5 @@
     </inertial>
     <visual>
-      <origin xyz="0.15096 0.021534 -0.267342" rpy="0 0 0"/>
+      <origin xyz="0.15096 -0.047 -0.267342" rpy="0 0 -0.37"/>
       <geometry>
         <mesh filename="package://robotic_arm/meshes/link3_part_1.stl" scale="${scale}"/>
@@ -80,5 +80,5 @@
     </visual>
     <collision>
-      <origin xyz="0.15096 0.021534 -0.267342" rpy="0 0 0"/>
+      <origin xyz="0.15096 -0.047 -0.267342" rpy="0 0 -0.37"/>
       <geometry>
         <mesh filename="package://robotic_arm/meshes/link3_part_1.stl" scale="${scale}"/>
@@ -92,5 +92,5 @@
   </joint>
   <joint name="Revolute_1" type="continuous">
-    <origin xyz="0.0 0.0 0.029" rpy="0 0 0"/>
+    <origin xyz="0.0 0.0 0.1" rpy="0 0 0"/>
     <parent link="base_link"/>
     <child link="Link_1_1"/>
@@ -99,16 +99,16 @@
   </joint>
   <joint name="Revolute_2" type="revolute">
-    <origin xyz="-0.016725 0.044458 0.22" rpy="0 0 0"/>
+    <origin xyz="0.0 0.044458 0.15" rpy="0 -0.1 0"/>
     <parent link="Link_1_1"/>
     <child link="link_2_1"/>
-    <axis xyz="0.352111 -0.935958 -0.0"/>
-    <limit upper="1.134464" lower="-4.014257" effort="50" velocity="5"/>
+    <axis xyz="0 1 0"/>
+    <limit upper="1.2" lower="-0.40" effort="50" velocity="5"/>
   </joint>
   <joint name="Revolute_3" type="revolute">
-    <origin xyz="-0.134235 -0.065992 0.018342" rpy="0 0 0"/>
+    <origin xyz="-0.150535 0.0 0.018342" rpy="0 -0.65 0"/>
     <parent link="link_2_1"/>
     <child link="link3_part_1"/>
-    <axis xyz="0.352111 -0.935958 -0.0"/>
-    <limit upper="1.48353" lower="0.0" effort="50" velocity="5"/>
+    <axis xyz="0 1 0"/>
+    <limit upper="0.8" lower="-0.3" effort="50" velocity="5"/>
   </joint>
   <gazebo>
@@ -142,8 +142,8 @@
 <!--
 Neutral Position of Robotic Arm
-ros2 topic pub /arm_controller/joint_trajectory trajectory_msgs/msg/JointTrajectory "
+ros2 topic pub -1 /arm_controller/joint_trajectory trajectory_msgs/msg/JointTrajectory "
 joint_names: ['Revolute_1', 'Revolute_2', 'Revolute_3']
 points:
 - positions: [-0.35, 0.2, 0.5]
-  time_from_start: {sec: 2} "
+  time_from_start: {sec: 2}"
 -->

Commit message: Did pick and place operation with voice api

File: robotic_arm/urdf/robotic.xacro (robot description, xacro)
@@ -169,5 +169,5 @@
     <child link="linktwo_1"/>
     <axis xyz="-1.0 0.0 0.0"/>
-    <limit upper="1.07" lower="-0.36" effort="100" velocity="100"/>
+    <limit upper="1.07" lower="-0.39" effort="100" velocity="100"/>
   </joint>
   <joint name="Revolute_3" type="revolute">
@@ -190,5 +190,5 @@
     <child link="gripper_right_1"/>
     <axis xyz="1.0 0.0 0.0"/>
-    <limit upper="0.07" lower="0.00" effort="500" velocity="5"/>
+    <limit upper="0.07" lower="0.00" effort="40" velocity="5"/>
   </joint>
   <joint name="Slider_2" type="prismatic">
@@ -197,5 +197,5 @@
     <child link="gripper_left_1"/>
     <axis xyz="-1.0 0.0 0.0"/>
-    <limit upper="0.07" lower="0.00" effort="500" velocity="5"/>
+    <limit upper="0.07" lower="0.00" effort="40" velocity="5"/>
     <mimic joint="Slider_1"/>
   </joint>
@@ -241,5 +241,7 @@
     <joint name="Slider_1">
       <command_interface name="position"/>
-      <state_interface name="position"/>
+      <state_interface name="position">
+        <param name="initial_value">0.06</param>
+      </state_interface>
       <state_interface name="velocity"/>
       <state_interface name="effort"/>
@@ -248,9 +250,17 @@
 </robot>
 <!--
-Neutral Position of Robotic Arm
+Place
 ros2 topic pub -1 /arm_controller/joint_trajectory trajectory_msgs/msg/JointTrajectory "
-joint_names: ['Revolute_1', 'Revolute_2', 'Revolute_3']
+joint_names: ['Revolute_1', 'Revolute_2', 'Revolute_3', 'Revolute_4']
 points:
-- positions: [0.0, 0.0, 0.0]
-  time_from_start: {sec: 2}"
+- positions: [-1.57, -0.4, 0.4, 1.2]
+  time_from_start: {sec: 3}"
 -->
+<!--
+Pick
+ros2 topic pub -1 /arm_controller/joint_trajectory trajectory_msgs/msg/JointTrajectory "
+joint_names: ['Revolute_1', 'Revolute_2', 'Revolute_3', 'Revolute_4']
+points:
+- positions: [-1.57, 0.4, 0.6, 0.5]
+  time_from_start: {sec: 3}"
+-->
